File: Power-Sense.kicad_sch (KiCad schematic)
At the start: 23 parts, among them U10 SN74LVC1G17DBVR, U9 INA228AIDGSR

Commit message: New UI
Other:
- note added: "Change to 200k"
Changed lines of the file:
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@@
+		)
+	)
+	(text "Change to 200k"
+		(exclude_from_sim no)
+		(at 81.026 102.108 0)
+		(effects
+			(font
+				(size 1.27 1.27)
+			)
 		)
 	)
