File: USB-PD.kicad_sch (KiCad schematic)
At the start: 63 parts, among them J2 61300411121, Q10 SQJB90EP-T1_GE3, Q11 AO3404A, Q8 AO3404A, Q9 AO3404A, U4 TPS26750SRSMR, U5 LM2765, U6 CAT24C512YI-GT3, U7 74LVC1G08SE-7, U8 LTC7004x

Commit message: Cleaned up the hierarchy
Parts:
- removed TP20: tp_round_70, TestPoint:TestPoint_Pad_1.5x1.5mm, symbol Connector:TestPoint
- TP14, TP15, TP16, TP17, TP18, TP19, TP21, TP22, TP23, TP24, TP25, TP26: footprint TestPoint:TestPoint_Pad_1.5x1.5mm -> TestPoint:TestPoint_Pad_D1.0mm
Connections:
- net +VBUS renamed VBUS
- net +VBUS_SENSED renamed VBUS_SENSED
Other:
- moved on the sheet: C38, C39, C40, C41, C42, C43, C44, C45, C46, C47, C48, C49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

Commit message: Starting with layout, oled, encoder, xt90
Connections:
- net GPIO14_R renamed I2CC_SCL_MCU
- net GPIO15_R renamed I2CC_SDA_MCU
Changed lines of the file:
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@@
 	)
 	(bus_entry
-		(at 163.83 154.94)
-		(size 2.54 2.54)
-		(stroke
-			(width 0)
-			(type default)
-		)
-	)
-	(bus_entry
 		(at 337.82 186.69)
 		(size 2.54 -2.54)
@@
 	)
 	(bus_entry
-		(at 81.28 228.6)
-		(size -2.54 -2.54)
+		(at 163.83 154.94)
+		(size 2.54 2.54)
 		(stroke
 			(width 0)
@@
 	(bus
 		(pts
-			(xy 166.37 157.48) (xy 168.91 157.48)
+			(xy 167.64 152.4) (xy 170.18 152.4)
 		)
 		(stroke
@@
 		)
 	)
-	(bus
-		(pts
-			(xy 66.04 214.63) (xy 77.47 214.63)
-		)
-		(stroke
-			(width 0)
-			(type default)
-		)
-	)
 	(wire
 		(pts
@@
 		)
 	)
+	(bus
+		(pts
+			(xy 166.37 160.02) (xy 166.37 154.94)
+		)
+		(stroke
+			(width 0)
+			(type default)
+		)
+	)
 	(wire
 		(pts
@@
 	(bus
 		(pts
-			(xy 166.37 157.48) (xy 166.37 160.02)
+			(xy 167.64 152.4) (xy 167.64 154.94)
 		)
 		(stroke
@@
 		)
 	)
-	(bus
-		(pts
-			(xy 78.74 228.6) (xy 78.74 226.06)
-		)
-		(stroke
-			(width 0)
-			(type default)
-		)
-	)
 	(wire
 		(pts
@@
 	(bus
 		(pts
-			(xy 78.74 226.06) (xy 78.74 223.52)
+			(xy 78.74 223.52) (xy 78.74 228.6)
 		)
 		(stroke
@@
 		)
 	)
+	(bus
+		(pts
+			(xy 166.37 154.94) (xy 167.64 154.94)
+		)
+		(stroke
+			(width 0)
+			(type default)
+		)
+	)
 	(wire
 		(pts
@@
 		)
 	)
+	(bus
+		(pts
+			(xy 66.04 214.63) (xy 77.47 214.63)
+		)
+		(stroke
+			(width 0)
+			(type default)
+		)
+	)
 	(wire
 		(pts
@@
 		)
 	)
-	(label "GPIO15_R"
+	(label "I2CC_SDA_MCU"
 		(at 163.83 154.94 180)
 		(effects
@@
 		)
 	)
-	(label "GPIO14_R"
+	(label "I2CC_SCL_MCU"
 		(at 163.83 157.48 180)
 		(effects
@@
 	(hierarchical_label "{I2C1}"
 		(shape bidirectional)
-		(at 168.91 157.48 0)
+		(at 170.18 152.4 0)
 		(effects
 			(font

Commit message: Finished layout
Parts:
- C40: footprint Capacitor_SMD:C_0603_1608Metric -> Capacitor_SMD:C_0402_1005Metric
Other:
- note removed: "Input Signals"
- note removed: "Output Signals"

Commit message: Started routing
Other:
- title: (none) -> Nitride-Nano
Changed lines of the file:
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@@
 	(generator_version "10.0")
 	(paper "A3")
+	(title_block
+		(title "Nitride-Nano")
+		(date "2026-05-07")
+		(rev "R1")
+	)
 	(text "USB Type-C® and USB PD Controller With Integrated Power Switches"
 		(exclude_from_sim no)

Commit message: Finished routing
Parts:
- removed TP23: tp_round_70, TestPoint:TestPoint_Pad_D1.0mm, symbol Connector:TestPoint
- JP11: footprint Altium_port:SolderJumper-3_P1.3mm_Bridged2Bar12_RoundedPad1.0x1.5mm -> Jumper:SolderJumper-3_P1.3mm_Bridged2Bar12_RoundedPad1.0x1.5mm
Changed lines of the file:
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@@
 	(wire
 		(pts
-			(xy 27.94 269.24) (xy 53.34 269.24)
-		)
-		(stroke
-			(width 0)
-			(type default)
-		)
-	)
-	(wire
-		(pts
 			(xy 161.29 129.54) (xy 58.42 129.54)
 		)
@@
 		)
 	)
-	(label "TS"
-		(at 27.94 269.24 0)
-		(effects
-			(font
-				(size 1.27 1.27)
-			)
-			(justify left bottom)
-		)
-	)
 	(label "SWITCH_EN"
 		(at 358.14 144.78 0)
@@
 			)
 		)
-		(property "Footprint" "Altium_port:SolderJumper-3_P1.3mm_Bridged2Bar12_RoundedPad1.0x1.5mm"
+		(property "Footprint" "Jumper:SolderJumper-3_P1.3mm_Bridged2Bar12_RoundedPad1.0x1.5mm"
 			(at 367.03 99.06 0)
 			(hide yes)
@@
 					(unit 1)
 				)
-			)
-		)
-	)
-	(symbol
-		(lib_id "Connector:TestPoint")
-		(at 53.34 269.24 270)
-		(unit 1)
-		(body_style 1)
-		(exclude_from_sim no)
-		(in_bom no)
-		(on_board yes)
-		(in_pos_files yes)
-		(dnp no)
-		(property "Reference" "TP23"
-			(at 58.42 269.24 90)
-			(show_name no)
-			(do_not_autoplace no)
-			(effects
-				(font
-					(size 1.27 1.27)
-				)
-				(justify left bottom)
-			)
-		)
-		(property "Value" "tp_round_70"
-			(at 49.53 267.97 0)
-			(hide yes)
-			(show_name no)
-			(do_not_autoplace no)
-			(effects
-				(font
-					(size 1.27 1.27)
-				)
-				(justify left bottom)
-			)
-		)
-		(property "Footprint" "TestPoint:TestPoint_Pad_D1.0mm"
-			(at 53.34 269.24 0)
-			(hide yes)
-			(show_name no)
-			(do_not_autoplace no)
-			(effects
-				(font
-					(size 1.27 1.27)
-				)
-			)
-		)
-		(property "Datasheet" ""
-			(at 53.34 269.24 0)
-			(hide yes)
-			(show_name no)
-			(do_not_autoplace no)
-			(effects
-				(font
-					(size 1.27 1.27)
-				)
-			)
-		)
-		(property "Description" "Test Point, Round, 0.7mm"
-			(at 53.34 269.24 0)
-			(hide yes)
-			(show_name no)
-			(do_not_autoplace no)
-			(effects
-				(font
-					(size 1.27 1.27)
-				)
-			)
-		)
-		(property "LCSC" ""
-			(at 53.34 269.24 0)
-			(hide yes)
-			(show_name no)
-			(do_not_autoplace no)
-			(effects
-				(font
-					(size 1.27 1.27)
-				)
-			)
-		)
-		(pin "1"
-		)
-		(instances
-			(project "nitride-nano"
-				(path "/aaad0350-e7db-44d5-b7ef-99e6416f6948/a05511eb-3c5e-4a0d-8491-3131eaddecdc"
-					(reference "TP23")
-					(unit 1)
-				)
