File: USB-PD.kicad_sch (KiCad schematic)
At the start: 61 parts, among them J2 61300411121, Q10 SQJB90EP-T1_GE3, Q11 AO3404A, Q8 AO3404A, Q9 AO3404A, U4 TPS26750SRSMR, U5 LM2765, U6 CAT24C512YI-GT3, U7 74LVC1G08SE-7, U8 LTC7004x

Commit message: Changed UI around a bit, and improved CV handling
Parts:
- added JP14: Jumper_2_Bridged, Jumper:SolderJumper-2_P1.3mm_Bridged_RoundedPad1.0x1.5mm, symbol Jumper:Jumper_2_Bridged
- JP4, JP6, JP8, JP9: footprint Altium_port:jumper_solder_2pad_no_40x40_20 -> Jumper:SolderJumper-2_P1.3mm_Open_RoundedPad1.0x1.5mm
Connections:
- net +3V3_LDO: now also JP14.2 (B)
- net I2CC_SCL_MCU: now also JP8.2 (B); no longer JP9.2 (B)
- net I2CC_SDA_MCU: now also JP9.2 (B); no longer JP8.2 (B)
- net SWITCH_EN_MANUAL: now also JP14.1 (A)
Changed lines of the file:
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@@
 	)
 	(junction
+		(at 270.51 135.89)
+		(diameter 0)
+		(color 0 0 0 0)
+	)
+	(junction
 		(at 78.74 92.71)
 		(diameter 0)
@@
 	)
 	(bus_entry
-		(at 163.83 154.94)
+		(at 171.45 154.94)
 		(size 2.54 2.54)
 		(stroke
@@
 	)
 	(bus_entry
-		(at 163.83 157.48)
+		(at 171.45 157.48)
 		(size 2.54 2.54)
 		(stroke
@@
 	(bus
 		(pts
-			(xy 167.64 152.4) (xy 170.18 152.4)
+			(xy 175.26 152.4) (xy 177.8 152.4)
 		)
 		(stroke
@@
 	(bus
 		(pts
-			(xy 166.37 160.02) (xy 166.37 154.94)
+			(xy 173.99 160.02) (xy 173.99 154.94)
 		)
 		(stroke
@@
 	(wire
 		(pts
-			(xy 148.59 157.48) (xy 163.83 157.48)
-		)
-		(stroke
-			(width 0)
-			(type default)
-		)
-	)
-	(wire
-		(pts
 			(xy 228.6 201.93) (xy 231.14 201.93)
 		)
@@
 	(wire
 		(pts
+			(xy 287.02 130.81) (xy 287.02 135.89)
+		)
+		(stroke
+			(width 0)
+			(type default)
+		)
+	)
+	(wire
+		(pts
 			(xy 308.61 129.54) (xy 311.15 129.54)
 		)
@@
 	(bus
 		(pts
-			(xy 167.64 152.4) (xy 167.64 154.94)
+			(xy 175.26 152.4) (xy 175.26 154.94)
 		)
 		(stroke
@@
 	(wire
 		(pts
+			(xy 287.02 135.89) (xy 283.21 135.89)
+		)
+		(stroke
+			(width 0)
+			(type default)
+		)
+	)
+	(wire
+		(pts
 			(xy 236.22 111.76) (xy 250.19 111.76)
 		)
@@
 	(wire
 		(pts
+			(xy 270.51 135.89) (xy 270.51 138.43)
+		)
+		(stroke
+			(width 0)
+			(type default)
+		)
+	)
+	(wire
+		(pts
 			(xy 27.94 264.16) (xy 53.34 264.16)
 		)
@@
 	(wire
 		(pts
+			(xy 171.45 154.94) (xy 148.59 154.94)
+		)
+		(stroke
+			(width 0)
+			(type default)
+		)
+	)
+	(wire
+		(pts
 			(xy 38.1 132.08) (xy 38.1 134.62)
 		)
@@
 	(wire
 		(pts
+			(xy 270.51 135.89) (xy 273.05 135.89)
+		)
+		(stroke
+			(width 0)
+			(type default)
+		)
+	)
+	(wire
+		(pts
 			(xy 68.58 134.62) (xy 68.58 137.16)
 		)
@@
 	(wire
 		(pts
+			(xy 148.59 157.48) (xy 171.45 157.48)
+		)
+		(stroke
+			(width 0)
+			(type default)
+		)
+	)
+	(wire
+		(pts
 			(xy 148.59 134.62) (xy 161.29 134.62)
 		)
@@
 	(bus
 		(pts
-			(xy 166.37 154.94) (xy 167.64 154.94)
+			(xy 173.99 154.94) (xy 175.26 154.94)
 		)
 		(stroke
@@
 	(wire
 		(pts
-			(xy 270.51 116.84) (xy 270.51 138.43)
+			(xy 270.51 116.84) (xy 270.51 135.89)
 		)
 		(stroke
@@
 	(wire
 		(pts
-			(xy 148.59 154.94) (xy 163.83 154.94)
-		)
-		(stroke
-			(width 0)
-			(type default)
-		)
-	)
-	(wire
-		(pts
 			(xy 231.14 204.47) (xy 231.14 201.93)
 		)
@@
 		)
 	)
-	(label "I2CC_SDA_MCU"
-		(at 163.83 154.94 180)
-		(effects
-			(font
-				(size 1.27 1.27)
-			)
-			(justify right bottom)
-		)
-	)
 	(label "LTC_GATE"
 		(at 358.14 87.63 0)
@@
 		)
 	)
-	(label "I2CC_SCL_MCU"
-		(at 163.83 157.48 180)
-		(effects
-			(font
-				(size 1.27 1.27)
-			)
-			(justify right bottom)
-		)
-	)
 	(label "I2C0_SDA"
 		(at 316.23 184.15 0)
@@
 		)
 	)
+	(label "I2CC_SDA_MCU"
+		(at 171.45 157.48 180)
+		(effects
+			(font
+				(size 1.27 1.27)
+			)
+			(justify right bottom)
+		)
+	)
 	(label "TS"
 		(at 363.22 127 180)
@@
 		)
 	)
+	(label "I2CC_SCL_MCU"
+		(at 171.45 154.94 180)
+		(effects
+			(font
+				(size 1.27 1.27)
+			)
+			(justify right bottom)
+		)
+	)
 	(label "I2CC_SDA"
 		(at 151.13 134.62 0)
@@
 	(hierarchical_label "{I2C1}"
 		(shape bidirectional)
-		(at 170.18 152.4 0)
+		(at 177.8 152.4 0)
 		(effects
 			(font
@@
 			)
 		)
-		(property "Footprint" "Altium_port:jumper_solder_2pad_no_40x40_20"
+		(property "Footprint" "Jumper:SolderJumper-2_P1.3mm_Open_RoundedPad1.0x1.5mm"
 			(at 143.51 134.62 0)
 			(hide yes)
@@
 			)
 		)
-		(property "Footprint" "Altium_port:jumper_solder_2pad_no_40x40_20"
+		(property "Footprint" "Jumper:SolderJumper-2_P1.3mm_Open_RoundedPad1.0x1.5mm"
 			(at 143.51 137.16 0)
 			(hide yes)
@@
 	)
 	(symbol
+		(lib_id "Jumper:Jumper_2_Bridged")
+		(at 278.13 135.89 0)
+		(unit 1)
+		(body_style 1)
+		(exclude_from_sim no)
+		(in_bom yes)
+		(on_board yes)
+		(in_pos_files yes)
+		(dnp no)
+		(fields_autoplaced yes)
+		(property "Reference" "JP14"
+			(at 278.13 130.81 0)
+			(show_name no)
+			(do_not_autoplace no)
+			(effects
+				(font
+					(size 1.27 1.27)
+				)
+			)
+		)
+		(property "Value" "Jumper_2_Bridged"
+			(at 278.13 133.35 0)
+			(show_name no)
+			(do_not_autoplace no)
+			(effects
+				(font
+					(size 1.27 1.27)
+				)
+			)
+		)
+		(property "Footprint" "Jumper:SolderJumper-2_P1.3mm_Bridged_RoundedPad1.0x1.5mm"
+			(at 278.13 135.89 0)
+			(hide yes)
+			(show_name no)
+			(do_not_autoplace no)
+			(effects
+				(font
+					(size 1.27 1.27)
+				)
+			)
+		)
+		(property "Datasheet" ""
+			(at 278.13 140.97 0)
+			(hide yes)
+			(show_name no)
+			(do_not_autoplace no)
+			(effects
+				(font
+					(size 1.27 1.27)
+				)
+			)
+		)
+		(property "Description" "Jumper, 2-pole, closed/bridged"
+			(at 278.13 143.51 0)
+			(hide yes)
+			(show_name no)
+			(do_not_autoplace no)
+			(effects
+				(font
+					(size 1.27 1.27)
+				)
+			)
+		)
+		(pin "2"
+		)
+		(pin "1"
+		)
+		(instances
+			(project "nitride-nano"
+				(path "/aaad0350-e7db-44d5-b7ef-99e6416f6948/a05511eb-3c5e-4a0d-8491-3131eaddecdc"
+					(reference "JP14")
+					(unit 1)
+				)
+			)
+		)
+	)
+	(symbol
 		(lib_id "power:GND")
 		(at 180.34 194.31 0)
@@
 	)
 	(symbol
+		(lib_id "power:+3V3")
+		(at 287.02 130.81 0)
+		(unit 1)
+		(body_style 1)
+		(exclude_from_sim no)
+		(in_bom yes)
+		(on_board yes)
+		(in_pos_files yes)
+		(dnp no)
+		(property "Reference" "#PWR0147"
+			(at 287.02 130.81 0)
+			(hide yes)
+			(show_name no)
+			(do_not_autoplace no)
+			(effects
+				(font
+					(size 1.27 1.27)
+				)
+			)
+		)
+		(property "Value" "+3V3_LDO"
+			(at 287.02 127 0)
+			(show_name no)
+			(do_not_autoplace no)
+			(effects
+				(font
+					(size 1.27 1.27)
+				)
+			)
+		)
+		(property "Footprint" ""
+			(at 287.02 130.81 0)
+			(show_name no)
+			(do_not_autoplace no)
+			(effects
+				(font
+					(size 1.27 1.27)
+				)
+			)
+		)
+		(property "Datasheet" ""
+			(at 287.02 130.81 0)
+			(show_name no)
+			(do_not_autoplace no)
+			(effects
+				(font
+					(size 1.27 1.27)
+				)
+			)
+		)
+		(property "Description" ""
+			(at 287.02 130.81 0)
+			(show_name no)
+			(do_not_autoplace no)
+			(effects
+				(font
+					(size 1.27 1.27)
+				)
+			)
+		)
+		(pin "1"
+		)
+		(instances
+			(project "nitride-nano"
+				(path "/aaad0350-e7db-44d5-b7ef-99e6416f6948/a05511eb-3c5e-4a0d-8491-3131eaddecdc"
+					(reference "#PWR0147")
+					(unit 1)
+				)
+			)
+		)
+	)
+	(symbol
 		(lib_id "Connector:TestPoint")
 		(at 140.97 250.19 270)
@@
 			)
 		)
-		(property "Footprint" "Altium_port:jumper_solder_2pad_no_40x40_20"
+		(property "Footprint" "Jumper:SolderJumper-2_P1.3mm_Open_RoundedPad1.0x1.5mm"
 			(at 143.51 157.48 0)
 			(hide yes)
@@
 			)
 		)
-		(property "Footprint" "Altium_port:jumper_solder_2pad_no_40x40_20"
+		(property "Footprint" "Jumper:SolderJumper-2_P1.3mm_Open_RoundedPad1.0x1.5mm"
 			(at 143.51 154.94 0)
 			(hide yes)
