File: nitride-nano.kicad_pcb (KiCad board)
At the start: 6 copper layers, 120 x 57 mm, 287 parts, among them J1 DX07S024JJ2R1300, J2 61300411121, J3 XT-90-M, J4 SWD, J5 SSD1306, J6 XT90-F, Q1 EPC2367, Q10 SQJB90EP-T1_GE3, Q11 AO3404A, Q12 HUASHUO HSBB0115, Q13 AO3404A, Q2 EPC2367, Q3 EPC2367, Q4 EPC2367, Q5 HUASHUO HSBB0115, Q6 AGM612AP, Q8 AO3404A, Q9 AO3404A, SW1 EC11E15244G1, U1 LT8390AIUFD-PBF, U10 SN74LVC1G17DBVR, U11 LMR16006XDDCR, U12 FT234XD, U2 STM32G474CEUx, U3 TPD4S480RUKR, U4 TPS26750SRSMR, U5 LM2765, U6 CAT24C512YI-GT3, U7 74LVC1G08SE-7, U8 LTC7004x, U9 INA228AIDGSR, Y1 8M

Commit message: 20A fuse
Parts:
- removed the REF** at (111.9, 101.1)
- removed the REF** at (45.2, 118.4)
- F1: value 10A -> 20A
