File: nitride-nano.kicad_pcb (KiCad board)
At the start: 6 copper layers, 120 x 57 mm, 315 parts, among them J1 DX07S024JJ2R1300, J2 61300411121, J3 XT-90-M, J4 SWD, J5 SSD1306, J6 XT90-F, Q1 EPC2367, Q10 SQJB90EP-T1_GE3, Q11 AO3404A, Q12 HUASHUO HSBB0115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

Commit message: Changed UI around a bit, and improved CV handling
Parts:
- R1: moved to B.Cu
