File: Converter.kicad_sch (KiCad schematic)
At the start: 75 parts, among them Q1 ${MFGPN}, Q2 ${MFGPN}, Q3 ${MFGPN}, Q4 ${MFGPN}, Q5 Q_PMOS, U1 LT8390AIUFD-PBF

Commit message: Cleaned up the hierarchy
Connections:
- net PWR_REG_OUT: now reaches C29.1, FB5.2, FB6.2, FB7.2, FB8.2
- net PWR_UNREG_IN: now reaches C6.1, FB1.1, FB2.1, FB3.1, FB4.1
- net CC Set renamed CC_Set
- net CV Set renamed CV_Set
Changed lines of the file:
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@@
+	)
+	(junction
+		(at 383.54 95.25)
+		(diameter 0)
+		(color 0 0 0 0)
 	)
 	(junction
@@
 	(wire
 		(pts
+			(xy 383.54 95.25) (xy 386.08 95.25)
+		)
+		(stroke
+			(width 0)
+			(type default)
+		)
+	)
+	(wire
+		(pts
 			(xy 201.93 166.37) (xy 201.93 168.91)
 		)
@@
 			(width 0)
 			(type default)
-		)
-	)
-	(label "CV Set"
-		(at 328.93 196.85 0)
-		(effects
-			(font
-				(size 1.27 1.27)
-			)
-			(justify left bottom)
 		)
 	)
@@
 		)
 	)
-	(label "CC Set"
-		(at 85.09 137.16 180)
-		(effects
-			(font
-				(size 1.27 1.27)
-			)
-			(justify right bottom)
-		)
-	)
 	(label "INTVCC"
 		(at 81.28 102.87 0)
@@
 		)
 	)
+	(hierarchical_label "CC_Set"
+		(shape input)
+		(at 85.09 137.16 180)
+		(effects
+			(font
+				(size 1.27 1.27)
+			)
+			(justify right)
+		)
+	)
+	(hierarchical_label "CV_Set"
+		(shape input)
+		(at 328.93 196.85 0)
+		(effects
+			(font
+				(size 1.27 1.27)
+			)
+			(justify left)
+		)
+	)
+	(hierarchical_label "PWR_UNREG_IN"
+		(shape input)
+		(at 43.18 27.94 180)
+		(effects
+			(font
+				(size 1.27 1.27)
+			)
+			(justify right)
+		)
+	)
+	(hierarchical_label "PWR_REG_OUT"
+		(shape output)
+		(at 386.08 95.25 0)
+		(effects
+			(font
+				(size 1.27 1.27)
+			)
+			(justify left)
+		)
+	)

Commit message: inductor, output fets
Parts:
- added Q12: HUASHUO HSBB0115, thommys-parts2:PRPAK-8_L3.0-W3.0-P0.65-BL-EP, symbol Device:Q_PMOS
- added R57: 3.3, Resistor_SMD:R_0402_1005Metric, symbol Device:R_Small
- D3, D4: footprint (none) -> PCM_JLCPCB:DFN2020-3_L2.0-W2.0-P0.65-BR-1
- L1: footprint (none) -> thommys-parts2:IND-SMD_SL1265-101M; JLC (none) -> C22463848
- Q5: value Q_PMOS -> HUASHUO HSBB0115; footprint (none) -> thommys-parts2:PRPAK-8_L3.0-W3.0-P0.65-BL-EP; JLC (none) -> C22359236
Connections:
- net LOADTG: now also R21.2, R57.2
- net at C27.1, C28.1, Q5.S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: now also Q12.S
- net at FB5.1, FB6.1, FB7.1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: now also Q12.D
- net at Q5.G, R22.2: no longer R21.2
- net ISMON renamed Curr_FB
- new net: Q12.G, R57.1

Commit message: Starting with layout, oled, encoder, xt90
Parts:
- removed C14: 100uF, symbol Device:C_Polarized
- C7: footprint (none) -> Capacitor_SMD:CP_Elec_10x12.6; JLC (none) -> C3274502
Changed lines of the file:
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@@
 	)
 	(junction
-		(at 316.23 63.5)
-		(diameter 0)
-		(color 0 0 0 0)
-	)
-	(junction
 		(at 293.37 110.49)
 		(diameter 0)
@@
 	(wire
 		(pts
-			(xy 316.23 63.5) (xy 334.01 63.5)
-		)
-		(stroke
-			(width 0)
-			(type default)
-		)
-	)
-	(wire
-		(pts
 			(xy 340.36 72.39) (xy 351.79 72.39)
 		)
@@
 	(wire
 		(pts
-			(xy 334.01 63.5) (xy 334.01 66.04)
-		)
-		(stroke
-			(width 0)
-			(type default)
-		)
-	)
-	(wire
-		(pts
 			(xy 335.28 99.06) (xy 335.28 95.25)
 		)
@@
 	(wire
 		(pts
-			(xy 334.01 73.66) (xy 334.01 74.93)
-		)
-		(stroke
-			(width 0)
-			(type default)
-		)
-	)
-	(wire
-		(pts
 			(xy 317.5 95.25) (xy 316.23 95.25)
 		)
@@
 	(symbol
 		(lib_id "power:GND")
-		(at 334.01 74.93 0)
-		(unit 1)
-		(body_style 1)
-		(exclude_from_sim no)
-		(in_bom yes)
-		(on_board yes)
-		(in_pos_files yes)
-		(dnp no)
-		(property "Reference" "#PWR021"
-			(at 334.01 81.28 0)
-			(hide yes)
-			(show_name no)
-			(do_not_autoplace no)
-			(effects
-				(font
-					(size 1.27 1.27)
-				)
-			)
-		)
-		(property "Value" "GND"
-			(at 334.01 78.486 0)
-			(show_name no)
-			(do_not_autoplace no)
-			(effects
-				(font
-					(size 1.27 1.27)
-				)
-			)
-		)
-		(property "Footprint" ""
-			(at 334.01 74.93 0)
-			(hide yes)
-			(show_name no)
-			(do_not_autoplace no)
-			(effects
-				(font
-					(size 1.27 1.27)
-				)
-			)
-		)
-		(property "Datasheet" ""
-			(at 334.01 74.93 0)
-			(hide yes)
-			(show_name no)
-			(do_not_autoplace no)
-			(effects
-				(font
-					(size 1.27 1.27)
-				)
-			)
-		)
-		(property "Description" "Power symbol creates a global label with name \"GND\" , ground"
-			(at 334.01 74.93 0)
-			(hide yes)
-			(show_name no)
-			(do_not_autoplace no)
-			(effects
-				(font
-					(size 1.27 1.27)
-				)
-			)
-		)
-		(pin "1"
-		)
-		(instances
-			(project "nitride-nano"
-				(path "/aaad0350-e7db-44d5-b7ef-99e6416f6948/f0962043-1aad-4f17-a8f7-b50910365543"
-					(reference "#PWR021")
-					(unit 1)
-				)
-			)
-		)
-	)
-	(symbol
-		(lib_id "power:GND")
 		(at 111.76 91.44 0)
 		(unit 1)
@@
 	)
 	(symbol
-		(lib_id "Device:C_Polarized")
-		(at 334.01 69.85 0)
-		(unit 1)
-		(body_style 1)
-		(exclude_from_sim no)
-		(in_bom yes)
-		(on_board yes)
-		(in_pos_files yes)
-		(dnp no)
-		(property "Reference" "C14"
-			(at 331.216 67.564 0)
-			(show_name no)
-			(do_not_autoplace no)
-			(effects
-				(font
-					(size 1.27 1.27)
-				)
-				(justify right)
-			)
-		)
-		(property "Value" "100uF"
-			(at 333.502 72.39 0)
-			(show_name no)
-			(do_not_autoplace no)
-			(effects
-				(font
-					(size 1.27 1.27)
-				)
-				(justify right)
-			)
-		)
-		(property "Footprint" ""
-			(at 334.9752 73.66 0)
-			(hide yes)
-			(show_name no)
-			(do_not_autoplace no)
-			(effects
-				(font
-					(size 1.27 1.27)
-				)
-			)
-		)
-		(property "Datasheet" ""
-			(at 334.01 69.85 0)
-			(hide yes)
-			(show_name no)
-			(do_not_autoplace no)
-			(effects
-				(font
-					(size 1.27 1.27)
-				)
-			)
-		)
-		(property "Description" "Polarized capacitor"
-			(at 334.01 69.85 0)
-			(hide yes)
-			(show_name no)
-			(do_not_autoplace no)
-			(effects
-				(font
-					(size 1.27 1.27)
-				)
-			)
-		)
-		(property "Field5" "63SXV100M"
-			(at 334.01 69.85 0)
-			(hide yes)
-			(show_name no)
-			(do_not_autoplace no)
-			(effects
-				(font
-					(size 1.27 1.27)
-				)
-			)
-		)
-		(property "Voltage" "100V"
-			(at 334.01 69.85 0)
-			(hide yes)
-			(show_name no)
-			(do_not_autoplace no)
-			(effects
-				(font
-					(size 1.27 1.27)
-				)
-			)
-		)
-		(pin "1"
-		)
-		(pin "2"
-		)
-		(instances
-			(project "nitride-nano"
-				(path "/aaad0350-e7db-44d5-b7ef-99e6416f6948/f0962043-1aad-4f17-a8f7-b50910365543"
-					(reference "C14")
-					(unit 1)
-				)
-			)
-		)
-	)
-	(symbol
 		(lib_id "Device:C_Small")
 		(at 139.7 82.55 0)
@@
 			)
 		)
-		(property "Footprint" ""
+		(property "Footprint" "Capacitor_SMD:CP_Elec_10x12.6"
 			(at 121.6152 46.99 0)
 			(hide yes)
@@
 			(at 120.65 43.18 0)
 			(hide yes)
+			(show_name no)
+			(do_not_autoplace no)
+			(effects
+				(font
+					(size 1.27 1.27)
+				)
+			)
+		)
+		(property "JLC" "C3274502"
+			(at 120.65 43.18 0)
+			(hide yes)

Commit message: Finished layout
Parts:
- removed C15, C27: 10uF, Capacitor_SMD:C_1210_3225Metric, symbol Device:C_Small
- added C85: 100n X7R 100V, Capacitor_SMD:C_0603_1608Metric, symbol 0_passives:C_0603
- added NT2: nt_2pad_20x20_20_60x20, Altium_port:NetTie-2_SMD_Pad0.5mm, symbol Device:NetTie_2
- added R72: 4.7k 1%, Resistor_SMD:R_0402_1005Metric, symbol 0_passives:R_0402
- added R73: 10k @25°C, Resistor_SMD:R_0402_1005Metric, symbol Device:Thermistor_NTC
- D3, D4: footprint PCM_JLCPCB:DFN2020-3_L2.0-W2.0-P0.65-BR-1 -> thommys-parts2:DFN2020-3_L2.0-W2.0-P0.65-BR-1; symbol Device:D_Schottky -> Thommys-parts2:D_Schottky_3
- R18, R9: footprint Resistor_SMD:R_1206_3216Metric -> Resistor_SMD:R_1210_3225Metric
Connections:
- net GND: now also D4.A, C85.2, NT2.2; no longer D4.2 (A)
- net at C24.2, D2.2 (A), L1.2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: now also D3.A; no longer D3.2 (A)
- net at C16.1, C17.1, C18.1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: now also D3.K; no longer D3.1 (K)
- net at C23.2, D1.2 (A), Q1.2 (S)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: now also D4.K; no longer D4.1 (K)
- new net: NT2.1, R73.2
- new net +3V3: R72.1
- new net TEMP_SENSE_CONV: C85.1, R72.2, R73.1
Other:
- note added: "Or Coilcraft: C6609502"
- note added: "TODO: Recalc shunts"

Commit message: Started routing
Parts:
- added D20: LED, LED_SMD:LED_0603_1608Metric, symbol Device:LED
- added R75, R87: 10k, Resistor_SMD:R_0402_1005Metric, symbol Device:R
- added R85, R86: 124k, Resistor_SMD:R_0402_1005Metric, symbol Device:R_Small
Connections:
- net GND: now also R75.1, R87.1
- net at FB5.1, FB6.1, FB7.1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: now also R85.1
- net at C28.1, Q12.S, Q5.S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: now also D20.2 (A)
- net Conv-Disable: now reaches R7.2, R8.1, U1.6 (EN/UVLO)
- new net: R85.2, R86.1
- new net: D20.1 (K), R75.2
- new net Vsense_REG_OUT: R86.2, R87.2
Other:
- title: (none) -> Nitride-Nano
- moved on the sheet: C29, FB5, FB6, FB7, FB8

Commit message: Finished routing
Connections:
- net Vref is gone; now on net VREF: R3.1
Changed lines of the file:
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@@
+		)
+	)
+	(label "VREF"
+		(at 104.14 194.31 180)
+		(effects
+			(font
+				(size 1.27 1.27)
+			)
+			(justify right bottom)
 		)
 	)
@@
 		)
 	)
-	(label "Vref"
-		(at 104.14 194.31 0)
-		(effects
-			(font
-				(size 1.27 1.27)
-			)
-			(justify left bottom)
-		)
-	)

Commit message: fixed pinout of cpu, added freecad file for the housing
Parts:
- R10: value 3.3 -> 0.5
- R12: value 6.2 -> 1.5
Connections:
- net GND: now also JP1.2 (C); no longer JP1.3 (B)
- net INTVCC: now also JP1.3 (B); no longer JP1.2 (C)
Other:
- note added: "5A standard limit"
- note added: "SSFM Off"
- note removed: "SSFM On"
Changed lines of the file:
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@@
 		)
 	)
+	(text "5A standard limit"
+		(exclude_from_sim no)
+		(at 80.01 148.082 0)
+		(effects
+			(font
+				(face "Comfortaa Light")
+				(size 1.27 1.27)
+			)
+		)
+	)
 	(text "5V standard output"
 		(exclude_from_sim no)
@@
 		)
 	)
-	(text "SSFM On"
+	(text "SSFM Off\n"
 		(exclude_from_sim no)
 		(at 77.978 176.784 0)
@@
 	(wire
 		(pts
-			(xy 72.39 181.61) (xy 71.12 181.61)
-		)
-		(stroke
-			(width 0)
-			(type default)
-		)
-	)
-	(wire
-		(pts
 			(xy 184.15 157.48) (xy 184.15 130.81)
 		)
@@
 	(wire
 		(pts
+			(xy 62.23 173.99) (xy 67.31 173.99)
+		)
+		(stroke
+			(width 0)
+			(type default)
+		)
+	)
+	(wire
+		(pts
 			(xy 88.9 102.87) (xy 88.9 106.68)
 		)
@@
 	(wire
 		(pts
-			(xy 60.96 175.26) (xy 60.96 173.99)
-		)
-		(stroke
-			(width 0)
-			(type default)
-		)
-	)
-	(wire
-		(pts
 			(xy 210.82 166.37) (xy 201.93 166.37)
 		)
@@
 	(wire
 		(pts
-			(xy 60.96 173.99) (xy 67.31 173.99)
-		)
-		(stroke
-			(width 0)
-			(type default)
-		)
-	)
-	(wire
-		(pts
 			(xy 328.93 95.25) (xy 335.28 95.25)
 		)
@@
 	(wire
 		(pts
-			(xy 72.39 177.8) (xy 72.39 181.61)
-		)
-		(stroke
-			(width 0)
-			(type default)
-		)
-	)
-	(wire
-		(pts
 			(xy 335.28 104.14) (xy 335.28 105.41)
 		)
@@
 	(wire
 		(pts
+			(xy 72.39 180.34) (xy 72.39 177.8)
+		)
+		(stroke
+			(width 0)
+			(type default)
+		)
+	)
+	(wire
+		(pts
 			(xy 231.14 71.12) (xy 241.3 71.12)
 		)
@@
 	)
 	(label "INTVCC"
+		(at 62.23 173.99 180)
+		(effects
+			(font
+				(size 1.27 1.27)
+			)
+			(justify right bottom)
+		)
+	)
+	(label "INTVCC"
 		(at 241.3 71.12 180)
 		(effects
@@
 		)
 	)
-	(label "INTVCC"
-		(at 71.12 181.61 180)
-		(effects
-			(font
-				(size 1.27 1.27)
-			)
-			(justify right bottom)
-		)
-	)
 	(label "VREF"
 		(at 68.58 129.54 180)
@@
 	(symbol
 		(lib_id "power:GND")
+		(at 72.39 180.34 0)
+		(unit 1)
+		(body_style 1)
+		(exclude_from_sim no)
+		(in_bom yes)
+		(on_board yes)
+		(in_pos_files yes)
+		(dnp no)
+		(property "Reference" "#PWR022"
+			(at 72.39 186.69 0)
+			(hide yes)
+			(show_name no)
+			(do_not_autoplace no)
+			(effects
+				(font
+					(size 1.27 1.27)
+				)
+			)
+		)
+		(property "Value" "GND"
+			(at 72.39 183.896 0)
+			(show_name no)
+			(do_not_autoplace no)
+			(effects
+				(font
+					(size 1.27 1.27)
+				)
+			)
+		)
+		(property "Footprint" ""
+			(at 72.39 180.34 0)
+			(hide yes)
+			(show_name no)
+			(do_not_autoplace no)
+			(effects
+				(font
+					(size 1.27 1.27)
+				)
+			)
+		)
+		(property "Datasheet" ""
+			(at 72.39 180.34 0)
+			(hide yes)
+			(show_name no)
+			(do_not_autoplace no)
+			(effects
+				(font
+					(size 1.27 1.27)
+				)
+			)
+		)
+		(property "Description" "Power symbol creates a global label with name \"GND\" , ground"
+			(at 72.39 180.34 0)
+			(hide yes)
+			(show_name no)
+			(do_not_autoplace no)
+			(effects
+				(font
+					(size 1.27 1.27)
+				)
+			)
+		)
+		(pin "1"
+		)
+		(instances
+			(project "nitride-nano"
+				(path "/aaad0350-e7db-44d5-b7ef-99e6416f6948/f0962043-1aad-4f17-a8f7-b50910365543"
+					(reference "#PWR022")
+					(unit 1)
+				)
+			)
+		)
+	)
+	(symbol
+		(lib_id "power:GND")
 		(at 119.38 204.47 0)
 		(unit 1)
@@
 			)
 		)
-		(property "Value" "6.2"
+		(property "Value" "1.5"
 			(at 281.94 153.67 90)
 			(show_name no)
@@
 			)
 		)
-		(property "Value" "3.3"
+		(property "Value" "0.5"
 			(at 190.5 127 90)
 			(show_name no)
@@
 	)
 	(symbol
-		(lib_id "power:GND")
-		(at 60.96 175.26 0)
-		(unit 1)
-		(body_style 1)
-		(exclude_from_sim no)
-		(in_bom yes)
-		(on_board yes)
-		(in_pos_files yes)
-		(dnp no)
-		(property "Reference" "#PWR037"
-			(at 60.96 181.61 0)
-			(hide yes)
-			(show_name no)
-			(do_not_autoplace no)
-			(effects
-				(font
-					(size 1.27 1.27)
-				)
-			)
-		)
-		(property "Value" "GND"
-			(at 60.96 178.816 0)
-			(show_name no)
-			(do_not_autoplace no)
-			(effects
-				(font
-					(size 1.27 1.27)
-				)
-			)
-		)
-		(property "Footprint" ""
-			(at 60.96 175.26 0)
-			(hide yes)
-			(show_name no)
-			(do_not_autoplace no)
-			(effects
-				(font
-					(size 1.27 1.27)
-				)
-			)
-		)
-		(property "Datasheet" ""
-			(at 60.96 175.26 0)
-			(hide yes)
-			(show_name no)
-			(do_not_autoplace no)
-			(effects
-				(font
-					(size 1.27 1.27)
-				)
-			)
-		)
-		(property "Description" "Power symbol creates a global label with name \"GND\" , ground"
-			(at 60.96 175.26 0)
-			(hide yes)
-			(show_name no)
-			(do_not_autoplace no)
-			(effects
-				(font
-					(size 1.27 1.27)
-				)
-			)
-		)
-		(pin "1"
-		)
-		(instances
-			(project "nitride-nano"
-				(path "/aaad0350-e7db-44d5-b7ef-99e6416f6948/f0962043-1aad-4f17-a8f7-b50910365543"
-					(reference "#PWR037")
-					(unit 1)
-				)
-			)
-		)
-	)
-	(symbol
 		(lib_id "Device:C_Small")
 		(at 119.38 200.66 0)
@@
 		(in_pos_files yes)
 		(dnp no)
-		(fields_autoplaced yes)
 		(property "Reference" "JP1"
 			(at 72.39 167.64 0)
