File: Converter.kicad_sch (KiCad schematic)
At the start: 83 parts, among them Q1 ${MFGPN}, Q12 HUASHUO HSBB0115, Q2 ${MFGPN}, Q3 ${MFGPN}, Q4 ${MFGPN}, Q5 HUASHUO HSBB0115, U1 LT8390AIUFD-PBF

Commit message: changed mistakes on board, first firmware version
Parts:
- R19: value 40k -> 357k; LCSC C137983 -> C27005
Other:
- note added: "36.7V standard output"
- note removed: "5V standard output"
Changed lines of the file:
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@@
 		)
 	)
-	(text "5V standard output"
+	(text "36.7V standard output"
 		(exclude_from_sim no)
-		(at 337.058 193.04 0)
+		(at 340.36 194.056 0)
 		(effects
 			(font
@@
 			)
 		)
-		(property "Value" "40k"
+		(property "Value" "357k"
 			(at 324.104 193.802 0)
 			(show_name no)
@@
 			)
 		)
-		(property "LCSC" "C137983"
+		(property "LCSC" "C27005"
 			(at 323.596 192.024 0)
 			(hide yes)

Commit message: New UI
Other:
- note added: "Change to allow for 12V input voltage that still enables CNV"
Changed lines of the file:
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@@
+		)
+	)
+	(text "Change to allow for 12V input voltage\n that still enables CNV"
+		(exclude_from_sim no)
+		(at 75.438 75.692 0)
+		(effects
+			(font
+				(face "Comfortaa Light")
+				(size 2 2)
+			)
 		)
 	)

Commit message: Changed UI around a bit, and improved CV handling
Parts:
- added R36: 10k, Resistor_SMD:R_0402_1005Metric, symbol Device:R_Small
Connections:
- net CV_Set: now also R36.2; no longer R19.2, R20.1, U1.16 (FB)
- net at FB5.1, FB6.1, FB7.1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: no longer R85.1
- net at C28.1, D20.2 (A), Q12.S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: now also R85.1
- new net: R19.2, R20.1, R36.1, U1.16 (FB)
Other:
- moved on the sheet: C28, Q12, Q5, R21, R22, R57
