File: nitride-nano.kicad_sch (KiCad schematic)
At the start: 13 parts, among them J3 XT-90-M, J6 XT90-F

Commit message: changed mistakes on board, first firmware version
Other:
- sheet MCU ports: added {I2C0}; removed none
Changed lines of the file:
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@@
 	)
 	(junction
+		(at 171.45 119.38)
+		(diameter 0)
+		(color 0 0 0 0)
+	)
+	(junction
 		(at 177.8 104.14)
 		(diameter 0)
@@
 		)
 	)
+	(bus
+		(pts
+			(xy 182.88 161.29) (xy 171.45 161.29)
+		)
+		(stroke
+			(width 0)
+			(type default)
+		)
+	)
 	(wire
 		(pts
@@
 	(bus
 		(pts
-			(xy 163.83 119.38) (xy 186.69 119.38)
+			(xy 163.83 119.38) (xy 171.45 119.38)
 		)
 		(stroke
@@
 		)
 	)
+	(bus
+		(pts
+			(xy 171.45 161.29) (xy 171.45 119.38)
+		)
+		(stroke
+			(width 0)
+			(type default)
+		)
+	)
 	(wire
 		(pts
@@
 		)
 	)
+	(bus
+		(pts
+			(xy 171.45 119.38) (xy 186.69 119.38)
+		)
+		(stroke
+			(width 0)
+			(type default)
+		)
+	)
 	(wire
 		(pts
@@
 			)
 		)
+		(pin "{I2C0}" bidirectional
+			(at 182.88 161.29 180)
+			(effects
+				(font
+					(size 1.27 1.27)
+				)
+				(justify left)
+			)
+		)
