File: PCB/Power-Sense.kicad_sch (KiCad schematic)
At the start: 23 parts, among them U10 SN74LVC1G17DBVR, U9 INA228AIDGSR

Commit message: Added NMOS output switch (rated for 20A this time)
Changed lines of the file:
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@@
 		(dnp no)
 		(property "Reference" "R56"
-			(at 278.765 132.08 90)
+			(at 281.686 126.746 90)
 			(show_name no)
 			(do_not_autoplace no)

Commit message: High current CC calibration
Other:
- note added: "Address: 1000000"
Changed lines of the file:
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@@
+		)
+	)
+	(text "Address: 1000000"
+		(exclude_from_sim no)
+		(at 177.292 147.32 0)
+		(effects
+			(font
+				(size 1.27 1.27)
+			)
 		)
 	)

Commit message: Preliminary finish of Rev3
Parts:
- removed C64: 100n X7R 100V, Capacitor_SMD:C_0603_1608Metric, symbol 0_passives:C_0603
- removed R55: 27R 1%, Resistor_SMD:R_0402_1005Metric, symbol 0_passives:R_0402
- removed R56: 4.7k 1%, Resistor_SMD:R_0402_1005Metric, symbol 0_passives:R_0402
- removed TP28, TP29: tp_round_70, TestPoint:TestPoint_Pad_D1.0mm, symbol Connector:TestPoint
- removed U10: SN74LVC1G17DBVR, Altium_port:sot25_95p_300x280x145_jedec_mo-178-aa_n, symbol 0_PD240W:SN74LVC1G17DBVR
- R60: value 8mR -> 3mR; JLC C46634461 -> C41382684; LCSC C46634461 -> C41382684
Connections:
- net INA_ALERT: no longer names the net of U9.3 (ALERT)
- no-connect marks 1 -> 0
