File: PCB/Power-Sense.kicad_sch (KiCad schematic)
At the start: 16 parts, among them U9 INA228AIDGSR

Commit message: Rev3 software now running and working. Couple hardware bugs being fixed for R4
Parts:
- removed R46: 100k, Resistor_SMD:R_0402_1005Metric, symbol Device:R_Small
Other:
- moved on the sheet: R44
Changed lines of the file:
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@@
-	)
-	(junction
-		(at 59.69 107.95)
-		(diameter 0)
-		(color 0 0 0 0)
 	)
 	(junction
@@
 	)
 	(junction
-		(at 59.69 99.06)
-		(diameter 0)
-		(color 0 0 0 0)
-	)
-	(junction
 		(at 59.69 116.84)
 		(diameter 0)
@@
 	(wire
 		(pts
-			(xy 54.61 105.41) (xy 54.61 107.95)
-		)
-		(stroke
-			(width 0)
-			(type default)
-		)
-	)
-	(wire
-		(pts
-			(xy 64.77 105.41) (xy 64.77 107.95)
-		)
-		(stroke
-			(width 0)
-			(type default)
-		)
-	)
-	(wire
-		(pts
-			(xy 59.69 83.82) (xy 59.69 99.06)
-		)
-		(stroke
-			(width 0)
-			(type default)
-		)
-	)
-	(wire
-		(pts
 			(xy 162.56 121.92) (xy 162.56 114.3)
 		)
@@
 	(wire
 		(pts
-			(xy 54.61 99.06) (xy 54.61 100.33)
+			(xy 59.69 83.82) (xy 59.69 100.33)
 		)
 		(stroke
@@
 	(wire
 		(pts
-			(xy 64.77 99.06) (xy 64.77 100.33)
-		)
-		(stroke
-			(width 0)
-			(type default)
-		)
-	)
-	(wire
-		(pts
 			(xy 193.04 142.24) (xy 194.31 142.24)
 		)
@@
 	(wire
 		(pts
-			(xy 54.61 107.95) (xy 59.69 107.95)
-		)
-		(stroke
-			(width 0)
-			(type default)
-		)
-	)
-	(wire
-		(pts
 			(xy 64.77 127) (xy 72.39 127)
 		)
@@
 	(wire
 		(pts
-			(xy 64.77 99.06) (xy 59.69 99.06)
-		)
-		(stroke
-			(width 0)
-			(type default)
-		)
-	)
-	(wire
-		(pts
 			(xy 195.58 121.92) (xy 195.58 109.22)
 		)
@@
 	(wire
 		(pts
-			(xy 59.69 107.95) (xy 59.69 110.49)
+			(xy 59.69 105.41) (xy 59.69 110.49)
 		)
 		(stroke
@@
 	(wire
 		(pts
-			(xy 59.69 107.95) (xy 64.77 107.95)
-		)
-		(stroke
-			(width 0)
-			(type default)
-		)
-	)
-	(wire
-		(pts
 			(xy 130.81 83.82) (xy 137.16 83.82)
-		)
-		(stroke
-			(width 0)
-			(type default)
-		)
-	)
-	(wire
-		(pts
-			(xy 54.61 99.06) (xy 59.69 99.06)
 		)
 		(stroke
@@
 	)
 	(symbol
-		(lib_id "Device:R_Small")
-		(at 64.77 102.87 0)
-		(mirror x)
-		(unit 1)
-		(body_style 1)
-		(exclude_from_sim no)
-		(in_bom yes)
-		(on_board yes)
-		(in_pos_files yes)
-		(dnp no)
-		(property "Reference" "R46"
-			(at 66.294 103.886 0)
-			(show_name no)
-			(do_not_autoplace no)
-			(effects
-				(font
-					(size 1.016 1.016)
-				)
-				(justify left)
-			)
-		)
-		(property "Value" "100k"
-			(at 65.786 102.108 0)
-			(show_name no)
-			(do_not_autoplace no)
-			(effects
-				(font
-					(size 1.27 1.27)
-				)
-				(justify left)
-			)
-		)
-		(property "Footprint" "Resistor_SMD:R_0402_1005Metric"
-			(at 64.77 102.87 0)
-			(hide yes)
-			(show_name no)
-			(do_not_autoplace no)
-			(effects
-				(font
-					(size 1.27 1.27)
-				)
-			)
-		)
-		(property "Datasheet" ""
-			(at 64.77 102.87 0)
-			(hide yes)
-			(show_name no)
-			(do_not_autoplace no)
-			(effects
-				(font
-					(size 1.27 1.27)
-				)
-			)
-		)
-		(property "Description" "Resistor, small symbol"
-			(at 64.77 102.87 0)
-			(hide yes)
-			(show_name no)
-			(do_not_autoplace no)
-			(effects
-				(font
-					(size 1.27 1.27)
-				)
-			)
-		)
-		(property "LCSC" "C60491"
-			(at 66.294 103.886 0)
-			(hide yes)
-			(show_name no)
-			(do_not_autoplace no)
-			(effects
-				(font
-					(size 1.27 1.27)
-				)
-			)
-		)
-		(pin "1"
-		)
-		(pin "2"
-		)
-		(instances
-			(project "nitride-nano"
-				(path "/aaad0350-e7db-44d5-b7ef-99e6416f6948/4379b8af-02d9-4f4c-b258-ce722d31539f"
-					(reference "R46")
-					(unit 1)
-				)
-			)
-		)
-	)
-	(symbol
 		(lib_id "0_PD240W:INA228AIDGSR")
 		(at 162.56 119.38 0)
@@
 	(symbol
 		(lib_id "Device:R_Small")
-		(at 54.61 102.87 0)
+		(at 59.69 102.87 0)
 		(mirror y)
 		(unit 1)
@@
 		(dnp no)
 		(property "Reference" "R44"
-			(at 53.086 101.854 0)
+			(at 58.166 101.854 0)
 			(show_name no)
 			(do_not_autoplace no)
@@
 		)
 		(property "Value" "100k"
-			(at 53.594 103.632 0)
+			(at 58.674 103.632 0)
 			(show_name no)
 			(do_not_autoplace no)
@@
 		)
 		(property "Footprint" "Resistor_SMD:R_0402_1005Metric"
-			(at 54.61 102.87 0)
+			(at 59.69 102.87 0)
 			(hide yes)
 			(show_name no)
@@
 		)
 		(property "Datasheet" ""
-			(at 54.61 102.87 0)
+			(at 59.69 102.87 0)
 			(hide yes)
 			(show_name no)
@@
 		)
 		(property "Description" "Resistor, small symbol"
-			(at 54.61 102.87 0)
+			(at 59.69 102.87 0)
 			(hide yes)
 			(show_name no)
@@
 		)
 		(property "LCSC" "C60491"
-			(at 53.086 101.854 0)
-			(hide yes)
-			(show_name no)
+			(at 58.166 101.854 0)
+			(hide yes)
+			(show_name no)
