File: PCB/Converter.kicad_sch (KiCad schematic)
At the start: 99 parts, among them Q1 ${MFGPN}, Q12 AO3400A, Q2 ${MFGPN}, Q3 ${MFGPN}, Q4 ${MFGPN}, Q5 ${MFGPN}, Q7 AO3401A, U1 LT8390AIUFD-PBF

Commit message: High current CC calibration
Connections:
- net VREF: no longer U1.8 (LOADEN)
- new net CNV-EN-LOADEN: U1.8 (LOADEN)
Changed lines of the file:
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@@
+	(wire
+		(pts
+			(xy 148.59 193.04) (xy 148.59 199.39)
+		)
+		(stroke
+			(width 0)
+			(type default)
+		)
+	)
 	(wire
 		(pts
@@
 		(pts
 			(xy 151.13 45.72) (xy 158.75 45.72)
+		)
+		(stroke
+			(width 0)
+			(type default)
+		)
+	)
+	(wire
+		(pts
+			(xy 148.59 199.39) (xy 147.32 199.39)
 		)
 		(stroke
@@
 	(label "INTVCC"
 		(at 67.31 111.76 0)
-		(effects
-			(font
-				(size 1.27 1.27)
-			)
-			(justify left bottom)
-		)
-	)
-	(label "VREF"
-		(at 148.59 193.04 0)
 		(effects
 			(font
@@
 		)
 	)
+	(hierarchical_label "CNV-EN-LOADEN"
+		(shape input)
+		(at 147.32 199.39 180)
+		(effects
+			(font
+				(size 1.27 1.27)
+			)
+			(justify right)
+		)
+	)

Commit message: Preliminary finish of Rev3
Parts:
- removed C1: 1nF, Capacitor_SMD:C_0402_1005Metric, symbol Device:C_Small
- removed C3: (no value), Capacitor_SMD:C_0402_1005Metric, symbol Device:C_Small
- removed R17: 10, Resistor_SMD:R_0402_1005Metric, symbol Device:R_Small
- removed R18: 0.002, Resistor_SMD:R_1206_3216Metric, symbol Device:R_Small
- removed R2: 18k, Resistor_SMD:R_0402_1005Metric, symbol Device:R_Small
- added C15: 1nF, Capacitor_SMD:C_0402_1005Metric, symbol Device:C_Small
- added C27: 100pF, Capacitor_SMD:C_0402_1005Metric, symbol Device:C_Small
- added C50: 10n X7R 100V, Capacitor_SMD:C_0402_1005Metric, symbol 0_passives:C_0402
- added C73: 100nF, Capacitor_SMD:C_0402_1005Metric, symbol Device:C_Small
- added R101: 1k, Resistor_SMD:R_0402_1005Metric, symbol Device:R_Small
- added U7: TMUX1574RSV, Package_DFN_QFN:UQFN-16_1.8x2.6mm_P0.4mm, symbol Analog_Switch:TMUX1574RSV
- C26: value 1uF -> 100pF; footprint Capacitor_SMD:C_0603_1608Metric -> Capacitor_SMD:C_0402_1005Metric; LCSC C23829972 -> (none); Voltage 100V -> (none)
- JP15: footprint Jumper:SolderJumper-2_P1.3mm_Open_RoundedPad1.0x1.5mm -> Jumper:SolderJumper-2_P1.3mm_Bridged_RoundedPad1.0x1.5mm
- R16: value 10 -> 18k; LCSC C25077 -> C25762
Connections:
- net +3V3: now also C73.1, U7.14 (VDD)
- net GND: now also C26.2, C15.2, C27.2, C50.2, C73.2, U7.13 (~{EN}), U7.6 (GND)
- net at C14.1, C16.1, C17.1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: now also C28.1, D20.2 (A), FB5.1, FB6.1, FB7.1, FB8.1, R19.1, R85.1; no longer R16.2
- net at U1.17 (VC): now also U7.7 (D3)
- net at C26.1, R16.1: now also U7.9 (S3A); no longer U1.11 (ISP)
- net ISN-L: now reaches U1.12 (ISN)
- net ISN-L: now also U7.5 (D2); no longer C26.2
- new net: C27.1, R101.2, U7.8 (S3B)
- new net: C50.1, R101.1
- new net: C15.1, R16.2
- new net High-Gain: U7.15 (SEL)
- new net IAMP-In: U7.1 (S1B)
- new net IAMP-Ref-In: U7.4 (S2B)
- new net ISN: U7.3 (S2A)
- new net ISP: U7.16 (S1A)
- new net ISP-L: U1.11 (ISP), U7.2 (D1)
- no-connect marks 0 -> 1

Commit message: Housing Rev3 added
Parts:
- removed TP35: tp_round_70, TestPoint:TestPoint_Pad_D1.0mm, symbol Connector:TestPoint
Changed lines of the file:
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@@
 	)
 	(junction
-		(at 127 207.01)
-		(diameter 0)
-		(color 0 0 0 0)
-	)
-	(junction
 		(at 127 204.47)
 		(diameter 0)
@@
 	(wire
 		(pts
-			(xy 127 210.82) (xy 127 207.01)
-		)
-		(stroke
-			(width 0)
-			(type default)
-		)
-	)
-	(wire
-		(pts
 			(xy 139.7 241.3) (xy 132.08 241.3)
 		)
@@
 	(wire
 		(pts
-			(xy 129.54 210.82) (xy 127 210.82)
-		)
-		(stroke
-			(width 0)
-			(type default)
-		)
-	)
-	(wire
-		(pts
 			(xy 311.15 104.14) (xy 311.15 199.39)
 		)
@@
 					(unit 1)
 				)
-			)
-		)
-	)
-	(symbol
-		(lib_id "Connector:TestPoint")
-		(at 129.54 210.82 270)
-		(unit 1)
-		(body_style 1)
-		(exclude_from_sim no)
-		(in_bom no)
-		(on_board yes)
-		(in_pos_files yes)
-		(dnp no)
-		(property "Reference" "TP35"
-			(at 134.62 210.82 90)
-			(show_name no)
-			(do_not_autoplace no)
-			(effects
-				(font
-					(size 1.27 1.27)
-				)
-				(justify left bottom)
-			)
-		)
-		(property "Value" "tp_round_70"
-			(at 125.73 209.55 0)
-			(hide yes)
-			(show_name no)
-			(do_not_autoplace no)
-			(effects
-				(font
-					(size 1.27 1.27)
-				)
-				(justify left bottom)
-			)
-		)
-		(property "Footprint" "TestPoint:TestPoint_Pad_D1.0mm"
-			(at 129.54 210.82 0)
-			(hide yes)
-			(show_name no)
-			(do_not_autoplace no)
-			(effects
-				(font
-					(size 1.27 1.27)
-				)
-			)
-		)
-		(property "Datasheet" ""
-			(at 129.54 210.82 0)
-			(hide yes)
-			(show_name no)
-			(do_not_autoplace no)
-			(effects
-				(font
-					(size 1.27 1.27)
-				)
-			)
-		)
-		(property "Description" "Test Point, Round, 0.7mm"
-			(at 129.54 210.82 0)
-			(hide yes)
-			(show_name no)
-			(do_not_autoplace no)
-			(effects
-				(font
-					(size 1.27 1.27)
-				)
-			)
-		)
-		(property "LCSC" ""
-			(at 129.54 210.82 0)
-			(hide yes)
-			(show_name no)
-			(do_not_autoplace no)
-			(effects
-				(font
-					(size 1.27 1.27)
-				)
-			)
-		)
-		(pin "1"
-		)
-		(instances
-			(project "nitride-nano"
-				(path "/aaad0350-e7db-44d5-b7ef-99e6416f6948/f0962043-1aad-4f17-a8f7-b50910365543"
-					(reference "TP35")
-					(unit 1)
-				)

Commit message: Rev3 software now running and working. Couple hardware bugs being fixed for R4
Parts:
- removed D11: BZT52C4V7S, PCM_JLCPCB:D_SOD-323, symbol PCM_JLCPCB-Diodes:Zener,BZT52C4V7S
- removed Q12: AO3400A, PCM_JLCPCB:Q_SOT-23, symbol PCM_JLCPCB-Transistors:NMOS,AO3400A
- removed Q5: ${MFGPN}, thommys-parts2:D1068, symbol Thommys-parts2:EPC2367
- removed Q7: AO3401A, PCM_JLCPCB:Q_SOT-23, symbol PCM_JLCPCB-Transistors:PMOS,AO3401A
- removed R21, R22: 100k, Resistor_SMD:R_0402_1005Metric, symbol Device:R_Small
- removed R57: 4.7k 1%, Resistor_SMD:R_0402_1005Metric, symbol 0_passives:R_0402
- removed R58: 27R 1%, Resistor_SMD:R_0402_1005Metric, symbol 0_passives:R_0402
Other:
- note removed: "Change to allow for 12V input voltage that still enables CNV"
- note removed: "TODO: 2uH is meer beter"
