File: PCB/nitride-nano.kicad_sch (KiCad schematic)
At the start: 13 parts, among them J3 XT-90-M, J6 XT90-F

Commit message: Revision 2; gate diodes, 5V into LT, i2c and uart lines fixed
Other:
- note removed: "TODO: SKEDD Conn instead of tagconnect"
Changed lines of the file:
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@@
-		)
-	)
-	(text "TODO: SKEDD Conn instead of tagconnect"
-		(exclude_from_sim no)
-		(at 306.07 197.612 0)
-		(effects
-			(font
-				(face "Comfortaa Medium")
-				(size 3 3)
-			)
 		)
 	)

Commit message: OLED Corruption fix, added UART Boot, DC-losses sim
Other:
- note added: "TODO: Inductor footprint too small"
- note removed: "TODO: Fix LV supply transient"
Changed lines of the file:
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@@
 		(company "Picobello B.V.")
 	)
-	(text "TODO: Fix LV supply transient"
+	(text "TODO: Inductor footprint too small"
 		(exclude_from_sim no)
-		(at 71.12 165.862 0)
+		(at 192.278 42.926 0)
 		(effects
 			(font
+				(face "Comfortaa Light")
 				(size 3 3)
 			)

Commit message: EPR sort of works with some chargers
Parts:
- removed R76: 10k, Resistor_SMD:R_0402_1005Metric, symbol Device:R
- added R76: 75k, Resistor_SMD:R_0402_1005Metric, symbol Device:R_Small
Connections:
- net GND: now also R76.2
- net at D21.1 (K): now also R76.1
Other:
- note added: "General TODO: ISMON not working I2C to PD chip not working Full efficiency sweep"
- note added: "HW TODO: Inductor footprint too small"
- note removed: "TODO: Inductor footprint too small"
Changed lines of the file:
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@@
 		(company "Picobello B.V.")
 	)
-	(text "TODO: Inductor footprint too small"
+	(text "HW TODO: Inductor footprint too small"
 		(exclude_from_sim no)
 		(at 192.278 42.926 0)
@@
 		)
 	)
+	(text "General TODO: \nISMON not working\nI2C to PD chip not working\nFull efficiency sweep\n"
+		(exclude_from_sim no)
+		(at 71.628 39.116 0)
+		(effects
+			(font
+				(face "Comfortaa Light")
+				(size 3 3)
+			)
+		)
+	)
 	(junction
 		(at 378.46 109.22)
@@
 	(wire
 		(pts
-			(xy 358.14 128.27) (xy 358.14 127)
+			(xy 358.14 125.73) (xy 358.14 128.27)
 		)
 		(stroke
@@
 	(wire
 		(pts
-			(xy 358.14 118.11) (xy 358.14 119.38)
+			(xy 358.14 118.11) (xy 358.14 120.65)
 		)
 		(stroke
@@
 	)
 	(symbol
-		(lib_id "Device:R")
-		(at 358.14 123.19 0)
-		(mirror x)
-		(unit 1)
-		(body_style 1)
-		(exclude_from_sim no)
-		(in_bom yes)
-		(on_board yes)
-		(in_pos_files yes)
-		(dnp no)
-		(fields_autoplaced yes)
-		(property "Reference" "R76"
-			(at 360.68 124.4601 0)
-			(show_name no)
-			(do_not_autoplace no)
-			(effects
-				(font
-					(size 1.27 1.27)
-				)
-				(justify left)
-			)
-		)
-		(property "Value" "10k"
-			(at 360.68 121.9201 0)
-			(show_name no)
-			(do_not_autoplace no)
-			(effects
-				(font
-					(size 1.27 1.27)
-				)
-				(justify left)
-			)
-		)
-		(property "Footprint" "Resistor_SMD:R_0402_1005Metric"
-			(at 356.362 123.19 90)
-			(hide yes)
-			(show_name no)
-			(do_not_autoplace no)
-			(effects
-				(font
-					(size 1.27 1.27)
-				)
-			)
-		)
-		(property "Datasheet" ""
-			(at 358.14 123.19 0)
-			(hide yes)
-			(show_name no)
-			(do_not_autoplace no)
-			(effects
-				(font
-					(size 1.27 1.27)
-				)
-			)
-		)
-		(property "Description" "Resistor"
-			(at 358.14 123.19 0)
-			(hide yes)
-			(show_name no)
-			(do_not_autoplace no)
-			(effects
-				(font
-					(size 1.27 1.27)
-				)
-			)
-		)
-		(property "LCSC" "C2906861"
-			(at 360.68 124.4601 0)
-			(hide yes)
-			(show_name no)
-			(do_not_autoplace no)
-			(effects
-				(font
-					(size 1.27 1.27)
-				)
-			)
-		)
-		(pin "2"
-		)
-		(pin "1"
-		)
-		(instances
-			(project "nitride-nano"
-				(path "/aaad0350-e7db-44d5-b7ef-99e6416f6948"
-					(reference "R76")
-					(unit 1)
-				)
-			)
-		)
-	)
-	(symbol
 		(lib_id "Graphic:Logo_Open_Hardware_Large")
 		(at 26.67 270.51 0)
@@
 					(unit 1)
 				)
+			)
+		)
+	)
+	(symbol
+		(lib_id "Device:R_Small")
+		(at 358.14 123.19 0)
+		(mirror y)
+		(unit 1)
+		(body_style 1)
+		(exclude_from_sim no)
+		(in_bom yes)
+		(on_board yes)
+		(in_pos_files yes)
+		(dnp no)
+		(property "Reference" "R76"
+			(at 356.616 122.174 0)
+			(show_name no)
+			(do_not_autoplace no)
+			(effects
+				(font
+					(size 1.016 1.016)
+				)
+				(justify left)
+			)
+		)
+		(property "Value" "75k"
+			(at 357.124 123.952 0)
+			(show_name no)
+			(do_not_autoplace no)
+			(effects
+				(font
+					(size 1.27 1.27)
+				)
+				(justify left)
+			)
+		)
+		(property "Footprint" "Resistor_SMD:R_0402_1005Metric"
+			(at 358.14 123.19 0)
+			(hide yes)
+			(show_name no)
+			(do_not_autoplace no)
+			(effects
+				(font
+					(size 1.27 1.27)
+				)
+			)
+		)
+		(property "Datasheet" ""
+			(at 358.14 123.19 0)
+			(hide yes)
+			(show_name no)
+			(do_not_autoplace no)
+			(effects
+				(font
+					(size 1.27 1.27)
+				)
+			)
+		)
+		(property "Description" "Resistor, small symbol"
+			(at 358.14 123.19 0)
+			(hide yes)
+			(show_name no)
+			(do_not_autoplace no)
+			(effects
+				(font
+					(size 1.27 1.27)
+				)
+			)
+		)
+		(property "LCSC" "C25798"
+			(at 356.616 122.174 0)
+			(hide yes)
+			(show_name no)
+			(do_not_autoplace no)
+			(effects
+				(font
+					(size 1.27 1.27)
+				)
+			)
+		)
+		(pin "1"
+		)
+		(pin "2"
+		)
+		(instances
+			(project "nitride-nano"
+				(path "/aaad0350-e7db-44d5-b7ef-99e6416f6948"
+					(reference "R76")
+					(unit 1)
+				)

Commit message: Added NMOS output switch (rated for 20A this time)
Connections:
- net GND: no longer D17.2, J3.1 (Pin_1)
- net Converter/PWR_REG_OUT renamed Converter/PWR_REG_OUT+
- new net Converter/PWR_REG_OUT-: D17.2, J3.1 (Pin_1)
Other:
- sheet Converter ports: added PWR_G, PWR_REG_OUT+, PWR_REG_OUT-; removed PWR_REG_OUT
- sheet MCU ports: added Turn_on_output; removed SWITCH_EN_MANUAL
- sheet USB-PD ports: added none; removed SWITCH_EN_MANUAL
- note added: "HW TODO: Inductor footprint too small EPC2361 output enable"
- note removed: "HW TODO: Inductor footprint too small"
- moved on the sheet: D21, R76

Commit message: High current CC calibration
Connections:
- net Converter/PWR_REG_OUT+: no longer D17.1, J3.2 (Pin_2)
- new net Power-Sense-Out/PWR-out: D17.1, J3.2 (Pin_2)
Other:
- sheet Power-Sense renamed Power-Sense-In
- added sheet Power-Sense-Out (Power-Sense-Out.kicad_sch)
- sheet Converter ports: added CNV-EN-LOADEN; removed none
- sheet MCU ports: added Converter-on-LOADEN; removed none
- note added: "General TODO: Full efficiency sweep"
- note added: "HW TODO:"
- note removed: "General TODO: ISMON not working I2C to PD chip not working Full efficiency sweep"
- note removed: "HW TODO: Inductor footprint too small EPC2361 output enable"
- moved on the sheet: D16, D17, D18, D21, F1, J3, J6, R30, R76

Commit message: Preliminary finish of Rev3
Parts:
- added F2: 20A, Fuse:Fuse_2512_6332Metric, symbol Device:Fuse
Connections:
- net Converter/PWR_REG_OUT+: now also F2.1; no longer D21.2 (A)
- net Converter/PWR_REG_OUT-: no longer D17.2, J3.1 (Pin_1)
- net Power-Sense-Out/PWR-out renamed Power-Sense-Out/Bus_V
- net Power-Sense-Out/Bus_V: now also D21.2 (A), F2.2
- new net Power-Sense-Out/PWR-In: D17.2, J3.1 (Pin_1)
Other:
- sheet Converter ports: added High-Gain, IAMP-In, IAMP-Ref-In, ISN, ISP; removed none
- sheet MCU ports: added Sel_high_gain; removed none
- sheet Power-Sense-In ports: added none; removed SWITCH_EN
- sheet Power-Sense-Out ports: added Bus_V, IAMP_Out, IAMP_Ref, ISN-Exp, ISP-Exp; removed none
- sheet USB-PD ports: added none; removed SWITCH_EN
- note added: "HW TODO: toggleable shunt amp?"
- note removed: "HW TODO:"
- moved on the sheet: D21, R76

Commit message: Rev3 software now running and working. Couple hardware bugs being fixed for R4
Connections:
- net Power-Sense-Out/PWR-In renamed OUTP-SW/PWR_REG_OUT-SW+
Other:
- added sheet OUTP-SW (OUTP.kicad_sch)
- sheet Converter ports: added none; removed PWR_G, PWR_REG_OUT-
- note added: "HW TODO: VREF Have 3v3 power the inamps shunt to lower side"
- note removed: "General TODO: Full efficiency sweep"
- note removed: "HW TODO: toggleable shunt amp?"
- moved on the sheet: D16, D17, D18, D21, F1, F2, J3, J6, R30, R76
